File: Schaltpläne/gesamt.brd (EAGLE design)
At the start: 100 x 80 mm, 9 parts, among them X1 332-02

Commit message: updated gesamten Schaltplan
Parts:
- moved SV2 168.1 mm to (88.9, 64.8), turned to 90 degrees
- moved R3 167.6 mm to (90.2, 43.2)
- moved R4 156.3 mm to (44.5, 74.5), turned to 180 degrees
- moved X1 148.3 mm to (22.6, 74.5), turned to 90 degrees
- moved R2 137.0 mm to (57.1, 43.2), turned to 180 degrees
- moved C1 119.4 mm to (43.2, 41.9), turned to 90 degrees
- moved R1 96.9 mm to (24.1, 39.4)
- moved SV1 90.0 mm to (25.4, 34.9), turned to 180 degrees
- moved MS1 89.5 mm to (12.7, 48.3)
Routing:
- net N$3: track 0.00 -> 219.3 mm
- net N$4: track 0.00 -> 161.9 mm
- net 3V: track 0.00 -> 149.1 mm
- net N$6: track 0.00 -> 73.4 mm
- net N$7: track 0.00 -> 72.3 mm
- net N$5: track 0.00 -> 37.4 mm
- net N$1: track 0.00 -> 23.7 mm
- net N$8: track 0.00 -> 21.7 mm
- net N$2: track 0.00 -> 20.8 mm
